File: pcb/ADB.kicad_pcb (KiCad board)
At the start: 2 copper layers, 77.2 x 50.8 mm, 54 parts, among them J1 Conn_01x10_Socket, J10 Conn_02x02_Counter_Clockwise, J11 Conn_02x02_Counter_Clockwise, J12 Conn_02x02_Counter_Clockwise, J13 Conn_02x02_Counter_Clockwise, J14 Conn_01x02_Socket, J15 Conn_01x04_Socket, J16 Conn_01x02_Socket, J17 Conn_01x02_Socket, J18 Conn_01x02_Socket, J19 Conn_01x03_Socket, J2 Conn_01x03_Pin, J20 Conn_01x03_Socket, J21 Conn_01x02_Socket, J22 Conn_01x02_Socket, J23 Conn_01x04_Socket, J24 Conn_01x02_Socket, J25 Conn_01x02_Socket, J26 Conn_01x02_Socket, J27 Conn_01x02_Socket, J28 Conn_01x02_Socket, J29 Conn_01x02_Socket, J3 Conn_01x08_Pin, J30 Conn_01x04_Socket, J31 Conn_01x02_Socket, J32 Conn_01x02_Socket, J33 Conn_01x02_Socket, J34 Conn_01x03_Socket, J35 Conn_01x03_Socket, J36 Conn_01x02_Socket, J37 Conn_01x02_Socket, J38 Conn_01x04_Socket, J39 Conn_01x02_Socket, J4 Conn_01x02_Pin, J40 Conn_01x02_Socket, J41 Conn_01x02_Socket, J42 Conn_01x02_Socket, J43 Conn_01x02_Socket, J5 Conn_01x10_Socket, J6 Conn_02x02_Counter_Clockwise, J7 Conn_02x02_Counter_Clockwise, J8 Conn_02x02_Counter_Clockwise, J9 Conn_02x02_Counter_Clockwise, U1 LM358

Commit message: Fix negative voltage descriptors
Connections:
- net VDD renamed VEE
Other:
- board text added: "VCC/VDD"
- board text added: "VEE/VSS"
- board text removed: "VCC"
- board text removed: "VDD"
Changed lines of the file:
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@@
   (net 1 "GND")
   (net 2 "VCC")
-  (net 3 "VDD")
+  (net 3 "VEE")
   (net 4 "Net-(J13-Pin_1)")
   (net 5 "Net-(J10-Pin_1)")
@@
       (net 1 "GND") (pinfunction "Pin_2") (pintype "passive"))
     (pad "3" thru_hole oval (at 0 5.08) (size 1.7 1.7) (drill 1) (layers "*.Cu" "*.Mask")
-      (net 3 "VDD") (pinfunction "Pin_3") (pintype "passive"))
+      (net 3 "VEE") (pinfunction "Pin_3") (pintype "passive"))
     (model "${KICAD6_3DMODEL_DIR}/Connector_PinHeader_2.54mm.3dshapes/PinHeader_1x03_P2.54mm_Vertical.wrl"
       (offset (xyz 0 0 0))
@@
       (stroke (width 0.1) (type solid)) (layer "F.Fab"))
     (pad "1" thru_hole rect (at 0 0 90) (size 1.7 1.7) (drill 1) (layers "*.Cu" "*.Mask")
-      (net 3 "VDD") (pinfunction "Pin_1") (pintype "passive"))
+      (net 3 "VEE") (pinfunction "Pin_1") (pintype "passive"))
     (pad "2" thru_hole oval (at 0 2.54 90) (size 1.7 1.7) (drill 1) (layers "*.Cu" "*.Mask")
-      (net 3 "VDD") (pinfunction "Pin_2") (pintype "passive"))
+      (net 3 "VEE") (pinfunction "Pin_2") (pintype "passive"))
     (pad "3" thru_hole oval (at 0 5.08 90) (size 1.7 1.7) (drill 1) (layers "*.Cu" "*.Mask")
-      (net 3 "VDD") (pinfunction "Pin_3") (pintype "passive"))
+      (net 3 "VEE") (pinfunction "Pin_3") (pintype "passive"))
     (pad "4" thru_hole oval (at 0 7.62 90) (size 1.7 1.7) (drill 1) (layers "*.Cu" "*.Mask")
-      (net 3 "VDD") (pinfunction "Pin_4") (pintype "passive"))
+      (net 3 "VEE") (pinfunction "Pin_4") (pintype "passive"))
     (pad "5" thru_hole oval (at 0 10.16 90) (size 1.7 1.7) (drill 1) (layers "*.Cu" "*.Mask")
-      (net 3 "VDD") (pinfunction "Pin_5") (pintype "passive"))
+      (net 3 "VEE") (pinfunction "Pin_5") (pintype "passive"))
     (pad "6" thru_hole oval (at 0 12.7 90) (size 1.7 1.7) (drill 1) (layers "*.Cu" "*.Mask")
-      (net 3 "VDD") (pinfunction "Pin_6") (pintype "passive"))
+      (net 3 "VEE") (pinfunction "Pin_6") (pintype "passive"))
     (pad "7" thru_hole oval (at 0 15.24 90) (size 1.7 1.7) (drill 1) (layers "*.Cu" "*.Mask")
-      (net 3 "VDD") (pinfunction "Pin_7") (pintype "passive"))
+      (net 3 "VEE") (pinfunction "Pin_7") (pintype "passive"))
     (pad "8" thru_hole oval (at 0 17.78 90) (size 1.7 1.7) (drill 1) (layers "*.Cu" "*.Mask")
-      (net 3 "VDD") (pinfunction "Pin_8") (pintype "passive"))
+      (net 3 "VEE") (pinfunction "Pin_8") (pintype "passive"))
     (pad "9" thru_hole oval (at 0 20.32 90) (size 1.7 1.7) (drill 1) (layers "*.Cu" "*.Mask")
-      (net 3 "VDD") (pinfunction "Pin_9") (pintype "passive"))
+      (net 3 "VEE") (pinfunction "Pin_9") (pintype "passive"))
     (pad "10" thru_hole oval (at 0 22.86 90) (size 1.7 1.7) (drill 1) (layers "*.Cu" "*.Mask")
-      (net 3 "VDD") (pinfunction "Pin_10") (pintype "passive"))
+      (net 3 "VEE") (pinfunction "Pin_10") (pintype "passive"))
     (model "${KICAD6_3DMODEL_DIR}/Connector_PinSocket_2.54mm.3dshapes/PinSocket_1x10_P2.54mm_Vertical.wrl"
       (offset (xyz 0 0 0))
@@
       (net 1 "GND") (pinfunction "Pin_1") (pintype "passive"))
     (pad "2" thru_hole oval (at 0 2.54) (size 1.7 1.7) (drill 1) (layers "*.Cu" "*.Mask")
-      (net 3 "VDD") (pinfunction "Pin_2") (pintype "passive"))
+      (net 3 "VEE") (pinfunction "Pin_2") (pintype "passive"))
     (model "${KICAD6_3DMODEL_DIR}/Connector_PinHeader_2.54mm.3dshapes/PinHeader_1x02_P2.54mm_Vertical.wrl"
       (offset (xyz 0 0 0))
@@
       (net 2 "VCC") (pintype "passive"))
     (pad "2" thru_hole circle (at 2.5 0 270) (size 1.6 1.6) (drill 0.8) (layers "*.Cu" "*.Mask")
-      (net 3 "VDD") (pintype "passive"))
+      (net 3 "VEE") (pintype "passive"))
     (model "${KICAD6_3DMODEL_DIR}/Capacitor_THT.3dshapes/CP_Radial_D6.3mm_P2.50mm.wrl"
       (offset (xyz 0 0 0))
@@
       (net 2 "VCC") (pintype "passive"))
     (pad "2" smd roundrect (at 1.475 0 270) (size 1.15 1.8) (layers "B.Cu" "B.Paste" "B.Mask") (roundrect_rratio 0.2173913043)
-      (net 3 "VDD") (pintype "passive"))
+      (net 3 "VEE") (pintype "passive"))
     (model "${KICAD6_3DMODEL_DIR}/Capacitor_SMD.3dshapes/C_1206_3216Metric.wrl"
       (offset (xyz 0 0 0))
@@
       (net 16 "Net-(J23-Pin_1)") (pinfunction "+") (pintype "input"))
     (pad "4" smd roundrect (at -2.475 -1.905 270) (size 1.95 0.6) (layers "B.Cu" "B.Paste" "B.Mask") (roundrect_rratio 0.25)
-      (net 3 "VDD") (pinfunction "V-") (pintype "power_in"))
+      (net 3 "VEE") (pinfunction "V-") (pintype "power_in"))
     (pad "5" smd roundrect (at 2.475 -1.905 270) (size 1.95 0.6) (layers "B.Cu" "B.Paste" "B.Mask") (roundrect_rratio 0.25)
       (net 23 "Net-(J38-Pin_1)") (pinfunction "+") (pintype "input"))
@@
     (effects (font (size 1.5 1.5) (thickness 0.2)))
   )
-  (gr_text "VDD" (at 185.42 121.92) (layer "F.SilkS")
+  (gr_text "VEE/VSS" (at 182.88 121.92) (layer "F.SilkS")
     (effects (font (size 1.5 1.5) (thickness 0.3) bold))
   )
@@
     (effects (font (size 1.5 1.5) (thickness 0.2)))
   )
-  (gr_text "VCC" (at 185.42 81.915) (layer "F.SilkS")
+  (gr_text "VCC/VDD" (at 185.42 81.915) (layer "F.SilkS")
     (effects (font (size 1.5 1.5) (thickness 0.3) bold))
   )
@@
     )
   )
-  (zone (net 3) (net_name "VDD") (layer "B.Cu") (hatch edge 0.5)
+  (zone (net 3) (net_name "VEE") (layer "B.Cu") (hatch edge 0.5)
     (priority 2)
     (connect_pads yes (clearance 0.254))
@@
     )
   )
-  (zone (net 3) (net_name "VDD") (layer "B.Cu") (hatch edge 0.5)
+  (zone (net 3) (net_name "VEE") (layer "B.Cu") (hatch edge 0.5)
     (priority 2)
     (connect_pads yes (clearance 0.254))

Commit message: Add gh-link
Other:
- board text added: "${link}"
Changed lines of the file:
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@@
+    (effects (font (size 1 1) (thickness 0.15)))
+  )
+  (gr_text "${link}" (at 216.916 101.6 90) (layer "F.SilkS")
     (effects (font (size 1 1) (thickness 0.15)))
   )
